File: Hardware/DIY/VisualightMicroDIY_032_gnd.sch (EAGLE design)
At the start: 27 parts, among them SW1 SPST_TACT-KMR2, U1 MIC5219 3.3V, U3 ATMEGA32U4, X2 USBPCB, Y1 16MHz

Commit message: Updates to firmware with MAC address and hardware with ground planes
Parts:
- renumbered U1 to 3.3VRREG, U3 to ATMEGA32U4
Other:
- note added: "3.3v REGULATOR"
- note added: "ATMEGA 32U4 CIRCUIT"
- note added: "BREAKOUT HEADER"
- note added: "ICSP SOCKET"
- note added: "POWER DECOUPLING"
- note added: "USB INTERFACE"
- note added: "WIFI"
- note added: "WIFI RESET SWITCH"
- moved on the sheet: C6, JP1, R1, R3, R5, R7, SW1, U$1
