File: Hardware/DIY/VisualightMicroDIY_036_gnd.brd (EAGLE design)
At the start: 49.5 x 34 mm, 30 parts, among them X2 USBPCB, Y1 16MHz

Commit message: SO MANY CHANGESgit commit -a -m
Parts:
- renumbered 3.3VRREG to 3.3VREG
