File: Hardware/DIY/SMD_cree_driver_led-mosfet002_dem.brd (EAGLE design)
At the start: 19.7 x 34 mm, 15 parts, among them Q1 BSS123, Q2 BSS123, Q3 BSS123, Q4 BSS123, Q5 NSI50350AST3G, Q6 NSI50350AST3G, Q7 NSI50350AST3G, Q8 NSI50350AST3G

Commit message: added board files
Parts:
- removed Q2, Q3: BSS123, transistor-small-signal:SOT23
- added U$2, U$5: NSI50350AST3G, on-semiconductor:SMC-2
- Q5, Q6: value NSI50350AST3G -> BSS123; device on-semiconductor:SMC-2 -> transistor-small-signal:SOT23
- moved Q5 16.5 mm to (26.9, 33.5), turned to 90 degrees
- moved Q6 8.39 mm to (21.6, 38.4), turned to 90 degrees
- renumbered Q7 to U$3, Q8 to U$4
Connections:
- net GND: now also U$2.C, U$5.C; no longer Q5.C, Q6.C
- net GREEN: now also Q6.1; no longer Q2.1
- net N$1: now also Q6.3; no longer Q2.3
- net N$12: now also U$5.A; no longer Q5.A
- net N$2: now also Q5.3; no longer Q3.3
- net N$4: now also Q6.2, U$2.A; no longer Q2.2, Q6.A
- net N$7: now also Q5.2; no longer Q3.2
- net RED: now also Q5.1; no longer Q3.1
Other:
- board text added: "DIY"
- board text added: "LED"
- board text added: "V 0.23"
- board text removed: "RGBW LED"
- board text removed: "V 0.24"
- board text removed: "blue"
- board text removed: "gnd"
- board text removed: "green"
- board text removed: "red"
- board text removed: "v0.24"
- board text removed: "vcc"
- board text removed: "white"
