File: Hardware/bulb/LED.brd (EAGLE design)
At the start: 100 x 80 mm, 9 parts, among them Q1 N-HEXFET_SOT323-, Q2 N-HEXFET_SOT323-, Q3 N-HEXFET_SOT323-

Commit message: lots of changes
Parts:
- removed SV1: (no value), con-lsta:FE05-1
- added IC1, IC2, IC3, IC4: LD117AV33, v-reg:TO220L1
- added JP1: (no value), adafruit:1X06
- added Q4: N-HEXFET_SOT323-, transistor-power:SOT223
- moved Q3 120.2 mm to (74.9, 52.1)
- moved Q2 104.5 mm to (80.0, 27.9)
- moved R4 96.8 mm to (81.3, 44.5), turned to 180 degrees
- moved R3 86.4 mm to (86.4, 17.8), turned to 180 degrees
- moved Q1 74.0 mm to (52.1, 29.2)
- moved R2 72.7 mm to (55.9, 44.5)
- moved R1 50.6 mm to (50.8, 17.8)
- moved U$1 20.4 mm to (67.3, 39.4)
Connections:
- removed net N$2: Q3.1, SV1.1
- removed net N$3: Q2.1, SV1.2
- removed net N$4: Q1.1, SV1.3
- new net BLUE: JP1.2, Q1.1
- new net GREEN: JP1.1, Q2.1
- new net N$10: Q2.4, U$1.6
- new net N$11: Q1.4, U$1.8
- new net N$12: Q4.4, U$1.2
- new net N$13: IC2.2, U$1.1
- new net N$14: IC3.2, U$1.7
- new net N$15: IC4.2, U$1.5
- new net N$16: IC1.2, U$1.3
- new net N$6: Q3.3, R4.2
- new net N$7: Q1.3, R1.2
- new net N$8: Q4.3, R2.2
- new net N$9: Q3.4, U$1.4
- new net RED: JP1.3, Q3.1
- new net WHITE: JP1.4, Q4.1
- net GND: now also IC1.1, IC2.1, IC3.1, IC4.1, JP1.5, R1.1, R2.1, R3.1, R4.1; no longer SV1.4
- net N$1: now also R3.2; no longer Q3.4
- net VCC: now also IC1.3, IC2.3, IC3.3, IC4.3, JP1.6; no longer SV1.5
Routing:
- net RED: track 0.00 -> 98.5 mm
- net GREEN: track 0.00 -> 64.8 mm
- net WHITE: track 0.00 -> 57.7 mm
- net N$15: track 0.00 -> 30.9 mm
- net GND: track 0.00 -> 25.5 mm, vias 0 -> 2
- net N$13: track 0.00 -> 23.2 mm
- net N$9: track 0.00 -> 20.9 mm
- net BLUE: track 0.00 -> 18.8 mm
- net N$16: track 0.00 -> 18.4 mm
- net N$12: track 0.00 -> 16.9 mm
- net N$10: track 0.00 -> 16.2 mm
- net N$11: track 0.00 -> 14.5 mm
- net N$14: track 0.00 -> 8.49 mm
- net N$7: track 0.00 -> 8.43 mm
- net N$1: track 0.00 -> 7.16 mm
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- added copper zone on layer 1, net GND
- added copper zone on layer 16, net VCC
Other:
- board size 100 x 80 mm -> 79.7 x 73.7 mm
- board text added: "+"
- board text added: "-"
- board text added: "B"
- board text added: "G"
- board text added: "R"
- board text added: "W"
