File: Hardware/bulb/10w_CREE_LED_driver.brd (EAGLE design)
At the start: 49 x 49 mm, 23 parts

Commit message: SO MANY CHANGESgit commit -a -m
Parts:
- moved U$1 8.51 mm to (24.5, 24.7)
Connections:
- removed net N$21: U$1.1
- removed net N$22: U$1.8
- removed net N$23: U$1.2
- removed net N$24: U$1.7
- removed net N$25: U$1.3
- removed net N$26: U$1.6
- removed net N$27: U$1.4
- removed net N$28: U$1.5
- net N$10: now also U$1.1
- net N$14: now also U$1.2
- net N$18: now also L1.1, U$1.6; no longer L4.1
- net N$19: now also L4.1, U$1.7; no longer L2.1
- net N$20: now also U$1.8
- net N$3: now also U$1.3
- net N$4: now also L2.1, U$1.5; no longer L1.1
- net N$6: now also U$1.4
Changed lines of the file:
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@@
 <plain>
 <circle x="24.5" y="24.5" radius="24.5" width="0.254" layer="20"/>
-<circle x="24.5" y="24.5" radius="3.625" width="0.4064" layer="45"/>
 </plain>
 <attributes>
@@
 <element name="D3" library="diode" package="DO214AC" value="SCHOTTKY" x="13.2" y="22.9" rot="R90"/>
 <element name="R8" library="adafruit" package="R0603" value="10K" x="8.2" y="13.5"/>
-<element name="U$1" library="led" package="CREE_XLAMP_XML" value="CREE_XLAMP_RGBW" x="17.1" y="28.9"/>
+<element name="U$1" library="led" package="CREE_XLAMP_XML" value="CREE_XLAMP_RGBW" x="24.5" y="24.7"/>
 </elements>
 <signals>
@@
 <wire x1="40.9838" y1="29.9" x2="39.2" y2="29.9" width="0.6096" layer="1"/>
 <wire x1="39.2" y1="29.9" x2="38.5" y2="29.2" width="0.6096" layer="1"/>
-</signal>
-<signal name="N$4">
-<contactref element="L1" pad="1"/>
+<contactref element="U$1" pad="3"/>
+<wire x1="26.65" y1="24.1" x2="38.5" y2="29.2" width="0" layer="19" extent="1-1"/>
 </signal>
 <signal name="N$5">
@@
 <wire x1="29.5" y1="9.4162" x2="29.5" y2="10.7" width="0.6096" layer="1"/>
 <wire x1="29.5" y1="10.7" x2="28.5" y2="11.7" width="0.6096" layer="1"/>
+<contactref element="U$1" pad="4"/>
+<wire x1="28.5" y1="11.7" x2="26.65" y2="22.7" width="0" layer="19" extent="1-1"/>
 </signal>
 <signal name="N$7">
@@
 <wire x1="22.7" y1="39" x2="23.1" y2="38.6" width="0.6096" layer="1"/>
 <wire x1="23.1" y1="38.6" x2="22.65" y2="38.15" width="0.6096" layer="1"/>
+<contactref element="U$1" pad="1"/>
+<wire x1="26.65" y1="26.7" x2="22.65" y2="38.15" width="0" layer="19" extent="1-1"/>
 </signal>
 <signal name="N$11">
@@
 <wire x1="7.7162" y1="18.2" x2="9.9" y2="18.2" width="0.6096" layer="1"/>
 <wire x1="9.9" y1="18.2" x2="10.7" y2="19" width="0.6096" layer="1"/>
+<contactref element="U$1" pad="2"/>
+<wire x1="10.7" y1="19" x2="26.65" y2="25.3" width="0" layer="19" extent="1-1"/>
 </signal>
 <signal name="N$15">
@@
 <contactref element="R8" pad="1"/>
 </signal>
+<signal name="N$4">
+<contactref element="L2" pad="1"/>
+<contactref element="U$1" pad="5"/>
+<wire x1="19.45" y1="8.7" x2="22.35" y2="22.7" width="0" layer="19" extent="1-1"/>
+</signal>
 <signal name="N$18">
+<contactref element="L1" pad="1"/>
+<contactref element="U$1" pad="6"/>
+<wire x1="22.35" y1="24.1" x2="41.9" y2="20.246" width="0" layer="19" extent="1-1"/>
+</signal>
+<signal name="N$19">
 <contactref element="L4" pad="1"/>
-</signal>
-<signal name="N$19">
-<contactref element="L2" pad="1"/>
+<contactref element="U$1" pad="7"/>
+<wire x1="6.9" y1="27.65" x2="22.35" y2="25.3" width="0" layer="19" extent="1-1"/>
 </signal>
 <signal name="N$20">
 <contactref element="L3" pad="1"/>
-</signal>
-<signal name="N$21">
-<contactref element="U$1" pad="1"/>
-</signal>
-<signal name="N$22">
 <contactref element="U$1" pad="8"/>
-</signal>
-<signal name="N$23">
-<contactref element="U$1" pad="2"/>
-</signal>
-<signal name="N$24">
-<contactref element="U$1" pad="7"/>
-</signal>
-<signal name="N$25">
-<contactref element="U$1" pad="3"/>
-</signal>
-<signal name="N$26">
-<contactref element="U$1" pad="6"/>
-</signal>
-<signal name="N$27">
-<contactref element="U$1" pad="4"/>
-</signal>
-<signal name="N$28">
-<contactref element="U$1" pad="5"/>
+<wire x1="22.35" y1="26.7" x2="33.15" y2="41.5" width="0" layer="19" extent="1-1"/>
 </signal>
 </signals>
