File: Hardware/bulb/10w_CREE_LED_driver.sch (EAGLE design)
At the start: 23 parts

Commit message: SO MANY CHANGESgit commit -a -m
Connections:
- removed net N$21: U$1.RA
- removed net N$22: U$1.RC
- removed net N$23: U$1.GA
- removed net N$24: U$1.GC
- removed net N$25: U$1.BA
- removed net N$26: U$1.BC
- removed net N$27: U$1.WA
- removed net N$28: U$1.WC
- net N$10: now also U$1.RA
- net N$14: now also U$1.GA
- net N$18: now also L1.1, U$1.BC; no longer L4.1
- net N$19: now also L4.1, U$1.GC; no longer L2.1
- net N$20: now also U$1.RC
- net N$3: now also U$1.BA
- net N$4: now also L2.1, U$1.WC; no longer L1.1
- net N$6: now also U$1.WA
Other:
- moved on the sheet: D2, D5, L2, L3, R3, R4, R5, R6, U$1
