File: Hardware/bulb/10w_LED_driver.brd (EAGLE design)
At the start: 49 x 49 mm, 23 parts

Commit message: SO MANY CHANGESgit commit -a -m
Parts:
- added R9: 330, SparkFun:0402-RES
- added TX: Green, SparkFun:LED-0603
- added X1: 52745-1090, con-molex:52745-1090
- added X2: USB-MICROB, SparkFun-Connectors:USB-MICROB
- moved R8 22.4 mm to (5.50, 35.7), turned to 90 degrees
- moved U$4 16.1 mm to (9.10, 35.6), turned to 180 degrees
- moved L4 12.7 mm to (15.0, 35.4), turned to 270 degrees
- moved R7 11.7 mm to (9.40, 31.6), turned to 180 degrees
- moved C1 10.6 mm to (23.2, 39.2), turned to 270 degrees
- moved R6 9.53 mm to (27.3, 44.9)
- moved D2 7.80 mm to (33.7, 33.1)
- moved L3 7.80 mm to (37.4, 38.5)
- moved R5 7.80 mm to (31.3, 35.6)
- moved U$3 7.80 mm to (31.4, 38.8)
- moved D3 6.20 mm to (13.2, 29.1), turned to 0 degrees
- moved C2 1.17 mm to (36.5, 12.2), turned to 90 degrees
- moved U$1 1.00 mm to (24.5, 24.5)
- moved R2 0.60 mm to (44.1, 33.4)
Connections:
- removed net N$13: R6.1
- removed net N$17: R8.1
- removed net N$9: R4.1
- new net D+IN: X1.7, X2.D+
- new net D-IN: X1.8, X2.D-
- new net D10: R8.1, X1.4
- new net D13: R4.1, X1.2
- new net D5: R6.1, X1.3
- new net D9: R2.1, X1.5
- new net TXLED: R9.1, X1.6
- new net UVCC: TX.A, X1.1, X2.VBUS
- net GND: now also X1.9, X2.GND
- net N$2: now also R9.2, TX.C; no longer R2.1
- net VCC: now also X1.10
Routing:
- net VCC: track 21.0 -> 114.4 mm, vias 0 -> 7
- net D9: track 0.00 -> 40.2 mm, vias 0 -> 2
- net D13: track 0.00 -> 36.8 mm, vias 0 -> 2
- net D5: track 0.00 -> 35.4 mm, vias 0 -> 2
- net UVCC: track 0.00 -> 19.7 mm, vias 0 -> 3
- net D10: track 0.00 -> 17.5 mm
- net D+IN: track 0.00 -> 13.4 mm
- net D-IN: track 0.00 -> 11.9 mm
- net N$20: track 17.3 -> 23.5 mm
- net N$14: track 16.4 -> 22.4 mm
- net N$12: track 0.00 -> 4.46 mm
- net TXLED: track 0.00 -> 4.34 mm
- net N$18: track 17.4 -> 14.1 mm
- net N$8: track 0.00 -> 2.98 mm
- net N$16: track 0.00 -> 2.87 mm
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- added copper zone on layer 1, net GND
