File: Hardware/bulb/VisualightMicroBulb_03.sch (EAGLE design)
At the start: 25 parts, among them U1 RN171RN171, X2 USB-MICROB, Y1 16MHz

Commit message: SO MANY CHANGESgit commit -a -m
Parts:
- added IC1, IC2: LD117AS25TR, v-reg:LD117AS25TR
- added R4: 2.2K, SparkFun:RESISTOR0402-RES
- added R8: 3.3K, SparkFun:RESISTOR0402-RES
- added U$1: U.FL, SparkFun-Connectors:U.FL
- added U2: SFW6R-3STE1LF, FCI_By_element14_Batch_1:SFW6R-3STE1LF
- added X1: 52745-1090, con-molex:52745-1090
Connections:
- new net ANT: U$1.SIGNAL, U1.ANT
- new net N$26: U2.6
- new net RAW: X1-7.S
- new net WIFIRESET: R4.2, R8.2, U1.RESET
- net +3V3_OUT: now also U1.VDD, U1.VDD_BATT, U1.VDD_RF
- net D+: now also X1-5.S
- net D-: now also X1-6.S
- net D10: now also U2.2, X1-2.S
- net D12: now also R4.1
- net D13: now also U2.1, X1-1.S
- net D5: now also U2.4, X1-4.S
- net D9: now also U2.3, X1-3.S
- net GND: now also R8.1, U$1.GND@0, U$1.GND@1, U1.GND@21, U1.GND@22, U1.GND@23, U1.GND@25, U1.GND@26, U1.GND@27, U2.5, X1-10.S, X1-9.S
- net UVCC: now also X1-8.S
- net WIFIDOUT: now also U1.TX
